File: hardware/flight-controller.kicad_sch (KiCad schematic)
At the start: 0 parts

Commit message: Saving KiCad Files and Updated Journal
Parts:
- added C1: 1uF, symbol Device:C
- added C10, C11, C12, C13, C2, C4, C6, C7, C8, C9: 10uF, symbol Device:C
- added C14, C16: 100nF, symbol Device:C
- added C15: 2.2 uF, symbol Device:C
- added C17, C18: 22uF, symbol Device:C
- added C3: 44uF, symbol Device:C
- added C5: 47nF, symbol Device:C
- added Card1: TF-01A, easyeda2kicad:TF-SMD_TF-01A, symbol easyeda2kicad:TF-01A
- added D1: LED, symbol Device:LED
- added J1: Screw_Terminal_01x02, symbol Connector:Screw_Terminal_01x02
- added L1: DFE252012F-1ROM=P2, symbol Device:L
- added L2: 1uH, symbol Device:L
- added L3: YHNR3015-5R6M, symbol Device:L
- added R1, R2: 5.1 K, symbol Device:R
- added R10: 5.23 K, symbol Device:R
- added R11, R12, R13, R3, R4, R5, R6, R8: 10K, symbol Device:R
- added R14: 100K, symbol Device:R
- added R15: 22.1K, symbol Device:R
- added R7: 383, symbol Device:R
- added R9: 30.1K, symbol Device:R
- added U1: TPS63070RNMR, easyeda2kicad:VQFN-15_L3.0-W2.5-P0.50-BL, symbol easyeda2kicad:TPS63070RNMR
- added U2: ICM-45686, easyeda2kicad:LGA-14_L3.0-W2.5-P0.50-TL, symbol easyeda2kicad:ICM-45686
- added U3: BQ25883RGER, easyeda2kicad:VFQFPN-24_L4.0-W4.0-P0.50-BL-EP2.8, symbol easyeda2kicad:BQ25883RGER
- added U4: BMP580, easyeda2kicad:LGA-10_L2.0-W2.0-P0.50-TL_BMP580, symbol easyeda2kicad:BMP580
- added U5: STM32F722RETx, Package_QFP:LQFP-64_10x10mm_P0.5mm, symbol MCU_ST_STM32F7:STM32F722RETx
- added U6: LMR51430, Package_TO_SOT_SMD:SOT-23-6, symbol Regulator_Switching:LMR51430
- added USB1: TYPE-C 16PIN 2MD, easyeda2kicad:USB-C-SMD_TYPE-C-16PIN-2MD-073, symbol easyeda2kicad:TYPE-C16PIN2MD
Connections:
- new net: R10.2, R8.1, R9.1, U3.7 (TS)
- new net: R1.1, USB1.B5 (CC2)
- new net: C2.1, L1.2, U3.21 (PMID), U3.22 (PMID)
- new net: D1.1 (K), U3.2 (STAT)
- new net: D1.2 (A), R6.2
- new net: C14.1, U1.3 (Vaux)
- new net: C16.2, L3.1, U6.2 (SW)
- new net: R14.2, R15.1, U6.4 (FB)
- new net: C16.1, U6.6 (CB)
- new net: C5.2, U3.12 (BTST)
- new net: R7.1, U3.8 (ILIM)
- new net: R2.1, USB1.A5 (CC1)
- new net: U5.18 (VSS), U5.31 (VSS), U5.47 (VSS), U5.63 (VSS)
- new net: L2.1, U1.9 (L2)
- new net: L2.2, U1.11 (L1)
- new net: R13.1, U1.2 (PG)
- new net: R12.1, U1.1 (PS/SYNC), U1.14 (EN)
- new net +3.3V: C17.1, C18.1, L3.2, R11.1, R14.1, R3.1, R4.1, R5.1, R6.1
- new net +5V: C10.1, C11.1, C12.1, C13.1, R13.2, U1.5 (FB), U1.7 (Vout)
- new net BAT+: C1.2, C14.2, C15.2, C17.2, C18.2, C2.2, C3.2, C4.1, C6.2, C7.2, C8.2, C9.2, J1.1 (Pin_1), J1.2 (Pin_2), R1.2, R15.2, R2.2, R7.2, R8.2, R9.2, U1.10 (PGND), U1.15 (Vsel), U1.4 (GND), U1.6 (FB2), U3.13 (BAT), U3.14 (BAT), U3.19 (GND), U3.20 (GND), U3.25 (EP), U6.1 (GND), USB1.13 (EH), USB1.14 (EH), USB1.A1B12 (GND), USB1.B1A12 (GND)
- new net BQ_CE: U3.3 (~{CE})
- new net BQ_INT: R5.2, U3.6 (~{INT})
- new net BQ_PG: R11.2, U3.9 (~{PG})
- new net BTST: C5.1, L1.1, U3.17 (SW), U3.18 (SW)
- new net Earth: C10.2, C11.2, C12.2, C13.2
- new net I2C_SCL: R4.2, U3.5 (SCL)
- new net I2C_SDA: R3.2, U3.4 (SDA)
- new net USB_DN: USB1.A7 (Dn1), USB1.B7 (Dn2)
- new net USB_DP: USB1.A6 (Dp1), USB1.B6 (Dp2)
- new net VBUS: C1.1, U3.23 (VBUS), USB1.A4B9 (VBUS), USB1.B4A9 (VBUS)
- new net VREGN: C6.1, R10.1, U3.11 (REGN)
- new net VSYS: C15.1, C3.1, C7.1, C8.1, C9.1, R12.2, U1.12 (Vin), U3.15 (SYS), U3.16 (SYS), U6.3 (VIN), U6.5 (EN)
- no-connect marks 0 -> 5

Commit message: KiCad updates and journal
Parts:
- added C19, C20, C21, C22: 100nF, symbol Device:C
- added R16, R17, R18, R19, R20, R21: 10K, symbol Device:R
Connections:
- net Earth is gone; now on net BAT+: C10.2, C11.2, C12.2, C13.2
- net +3.3V: now also Card1.4 (VDD), U2.5 (VDDIO), U2.8 (VDD), U4.1 (VDDIO), U4.10 (VDD), C19.2, C20.1, C21.1, C22.1, R16.1, R17.1, R18.1, R19.1, R20.1, R21.1
- net BAT+: now also Card1.10 (GND), Card1.11 (GND), Card1.12 (GND), Card1.13 (GND), Card1.6 (VSS), U2.6 (GND), U4.3 (VSS), U4.5 (SDO), U4.6 (CSB), U4.8 (VSS), U4.9 (VSS), C19.1, C20.2, C21.2, C22.2
- net BMP_SCK: now reaches U4.2 (SCK)
- net BMP_SDI: now reaches U4.4 (SDI)
- net BMP_INT: now reaches U4.7 (INT)
- net ICM_SDO: now reaches U2.1 (AP_SDO/AP_AD0)
- net ICM_INT1: now reaches U2.4 (INT1/INT)
- net SD_DAT2: now reaches Card1.1 (DAT2(RSV))
- net SD_DAT2: now also R18.2
- net SD_DAT3: now reaches Card1.2 (CDDAT3(CS))
- net SD_DAT3: now also R19.2
- net SD_CMD: now reaches Card1.3 (CMD(DI))
- net SD_CMD: now also R20.2
- net SD_CLK: now reaches Card1.5 (CLK(SCLK))
- net SD_CLK: now also R21.2
- net SD_DAT0: now reaches Card1.7 (DAT0(D0))
- net SD_DAT0: now also R16.2
- net SD_DAT1: now reaches Card1.8 (DAT1(RSV))
- net SD_DAT1: now also R17.2
- net SD_CD: now reaches Card1.9 (CD)
- no-connect marks 5 -> 10
Other:
- moved on the sheet: C10, C11, C12, C13, C14, C15, C16, C17, C18, C7, C8, C9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
